Commit message: gazeboo

File: description/robot.urdf.xacro (robot description, xacro)
@@ -3,3 +3,4 @@
     <xacro:include filename="robot_core.xacro"/>
     <!-- <xacro:include filename="inertial_macros.xacro"/> -->
+    <xacro:include filename="gazebo_control.xacro"/>
 </robot>

File: description/robot_core.xacro (robot description, xacro)
@@ -19,5 +19,5 @@
     </link>
     <!-- chassis -->
-    <joint name="chassis_joiny" type="fixed">
+    <joint name="chassis_joint" type="fixed">
         <parent link="base_link"/>
         <child link="chassis"/>
@@ -43,4 +43,7 @@
         </xacro:inertial_box>
     </link>
+    <gazebo reference="chassis">
+        <material>Gazebo/White</material>
+    </gazebo>
     <!-- left wheel -->
     <joint name="left_wheel_joint" type="continuous">
@@ -76,4 +79,7 @@
         </xacro:inertial_cylinder>
     </link>
+    <gazebo reference="left_wheel">
+        <material>Gazebo/Blue</material>
+    </gazebo>
     <!-- right wheel -->
     <joint name="right_wheel_joint" type="continuous">
@@ -109,4 +115,7 @@
         </xacro:inertial_cylinder>
     </link>
+    <gazebo reference="right_wheel_link">
+        <material>Gazebo/Blue</material>
+    </gazebo>
     <!-- caster wheel -->
     <joint name="caster_wheel_joint" type="fixed">
@@ -132,3 +141,8 @@
         </xacro:inertial_sphere>
     </link>
+    <gazebo reference="caster_wheel">
+        <material>Gazebo/Black</material>
+        <mu1 value="0.001" />
+        <mu2 value="0.001" />
+    </gazebo>
 </robot>
